File: hardware/HAT/PlanktoscopeHat-v0.1-fab.brd (EAGLE design)
At the start: 65 x 100 mm, 90 parts, among them K1 PINHD-2X20, P4 MA08-1, P5 MA08-1, P6 MA02-1, P7 MA08-1, P8 MA08-1, P9 MA02-1, Q1 5.8A/30V/35mΩ, Q2 DMG2305UX, Q3 DMP3013SFV-7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

Commit message: Hardware: BOM Addition and schematic update
Parts:
- C20: value 1uF -> 1µF
- R11: value 500R -> 499R
- R12: value 5k -> 4.99k
Changed lines of the file:
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@@
 <attribute name="VALUE" x="43.4125" y="84.73" size="1" layer="27" font="vector" ratio="12" align="center"/>
 </element>
-<element name="C20" library="microbuilder" library_urn="urn:adsk.eagle:library:18156183" package="_0805MP" package3d_urn="urn:adsk.eagle:package:18156346/1" value="1uF" x="48" y="89" smashed="yes" rot="R90">
+<element name="C20" library="microbuilder" library_urn="urn:adsk.eagle:library:18156183" package="_0805MP" package3d_urn="urn:adsk.eagle:package:18156346/1" value="1µF" x="48" y="89" smashed="yes" rot="R90">
 <attribute name="NAME" x="48.5" y="92.5" size="1" layer="25" font="vector" ratio="12" rot="R90" align="center"/>
 <attribute name="VALUE" x="49.27" y="87.4125" size="1" layer="27" font="vector" ratio="12" rot="R90" align="center"/>
@@
 <attribute name="VENDOR" value="JST" x="32" y="94" size="1.778" layer="27" rot="R180" display="off"/>
 </element>
-<element name="R11" library="microbuilder" library_urn="urn:adsk.eagle:library:18156183" package="_0805MP" package3d_urn="urn:adsk.eagle:package:18156346/1" value="500R" x="26" y="4" smashed="yes" rot="R270">
+<element name="R11" library="microbuilder" library_urn="urn:adsk.eagle:library:18156183" package="_0805MP" package3d_urn="urn:adsk.eagle:package:18156346/1" value="499R" x="26" y="4" smashed="yes" rot="R270">
 <attribute name="NAME" x="26" y="1.5" size="1" layer="25" font="vector" ratio="12" align="center"/>
 <attribute name="VALUE" x="24.73" y="5.5875" size="1" layer="27" font="vector" ratio="12" rot="R270" align="center"/>
 </element>
-<element name="R12" library="microbuilder" library_urn="urn:adsk.eagle:library:18156183" package="_0805MP" package3d_urn="urn:adsk.eagle:package:18156346/1" value="5k" x="28" y="4" smashed="yes" rot="R270">
+<element name="R12" library="microbuilder" library_urn="urn:adsk.eagle:library:18156183" package="_0805MP" package3d_urn="urn:adsk.eagle:package:18156346/1" value="4.99k" x="28" y="4" smashed="yes" rot="R270">
 <attribute name="NAME" x="29.5" y="4" size="1" layer="25" font="vector" ratio="12" rot="R90" align="center"/>
 <attribute name="VALUE" x="26.73" y="5.5875" size="1" layer="27" font="vector" ratio="12" rot="R270" align="center"/>
@@
 <element name="D3" library="OPL_Discrete_Semiconductor" library_urn="urn:adsk.eagle:library:8004488" package="SOD-123" package3d_urn="urn:adsk.eagle:package:8004543/1" value="40V-500MA" x="21" y="67" smashed="yes" rot="R180">
 <attribute name="MPN" value="B0540W" x="21" y="67" size="1.778" layer="27" rot="R180" display="off"/>
+<attribute name="NAME" x="21.889" y="67.635" size="0.381" layer="33" ratio="10" rot="R180"/>
 <attribute name="NAME" x="17.5" y="67" size="1" layer="25" font="vector" ratio="12" rot="R180" align="center"/>
-<attribute name="NAME" x="21.889" y="67.635" size="0.381" layer="33" ratio="10" rot="R180"/>
 <attribute name="VALUE" x="22.905" y="69.032" size="1" layer="27" font="vector" ratio="12" rot="R180" align="center"/>
 </element>
@@
 <element name="D4" library="OPL_Discrete_Semiconductor" library_urn="urn:adsk.eagle:library:8004488" package="SOD-123" package3d_urn="urn:adsk.eagle:package:8004543/1" value="40V-500MA" x="35" y="68" smashed="yes" rot="R180">
 <attribute name="MPN" value="B0540W" x="55" y="53" size="1.778" layer="27" rot="R180" display="off"/>
+<attribute name="NAME" x="35.889" y="68.635" size="0.381" layer="33" ratio="10" rot="R180"/>
 <attribute name="NAME" x="31.5" y="68" size="1" layer="25" font="vector" ratio="12" rot="R180" align="center"/>
-<attribute name="NAME" x="35.889" y="68.635" size="0.381" layer="33" ratio="10" rot="R180"/>
 <attribute name="VALUE" x="36.905" y="70.032" size="1" layer="27" font="vector" ratio="12" rot="R180" align="center"/>
 </element>
