File: hardware/HAT/PlanktoscopeHat-v1.0-fab.sch (EAGLE design)
At the start: 86 parts, among them J1 JUMPER-SMT_3_1-NC_PASTE_SILK, J2 JUMPER-SMT_3_1-NC_PASTE_SILK, J3 JUMPER-SMT_2_NC_PASTE_SILK, K1 SSQ-120-04-T-D, Q1 600mA/40V, Q2 DMG2305UX, Q3 DMP3013SFV-7, Q4 600mA/40V, U1 M24C32-WMN6, U2 LM36011YKBR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

Commit message: hardware: hat fab files
(cherry picked from commit 8a2ba7d7322f03550dc010669ea8b1d036b7b47b)
Parts:
- C19: value 10uF -> 100nF
- C20: value 100nF -> 10uF
- R11: value 10R -> 510R
- R12: value 1k -> 5.1k
Connections:
- removed net N$5: STROBE.TP, U2.STROBE
- net GPIO22: now also STROBE.TP, U2.STROBE
Other:
- note removed: "Target frequency: 25kHz for Noctua fan"
- moved on the sheet: +5V, C10, C11, C12, C13, C14, C15, C16, C17, C18, C19, C20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
